File: kicad/rosalyn-tx.kicad_pcb (KiCad board)
At the start: 4 copper layers, 56.6 x 41.1 mm, 38 parts, among them J1 USB-C, J2 SWD, J3 TURNIGY 9X, J4 Serial1, J5 Serial2, U1 SPX3819, U2 XC6206, U3 STM32F072C8, U4 E22-EBYTE, U5 SRV05-4

Commit message: added led drivers
Connections:
- net e22_busy renamed radio_busy
- net e22_dio1 renamed radio_dio1
- net e22_dio2 renamed radio_dio2
- net e22_nrst renamed radio_nrst
- net e22_nss renamed radio_nss
- net e22_rxen renamed radio_rxen
- net e22_txen renamed radio_txen
- net hmi_error1 renamed hmi_error
- net hmi_error2 renamed hmi_error_ext
- net hmi_status1 renamed hmi_status
- net hmi_status2 renamed hmi_status_ext
- J1 pad S1: GND -> Net-(J1-PadS1)
Routing:
- net Net-(J1-PadS1): track 0.00 -> 18.7 mm
- net GND: track 68.4 -> 59.4 mm
